File: extras/schematics/lora_tracker.sch (KiCad schematic (older format))
At the start: 18 parts, among them J1 Conn_Coaxial, J2 Conn_01x10_Female, J3 Conn_01x12_Female, J4 Conn_01x03_Female, U1 ESP32, U2 E22-400M30S, U3 Ai-Thinker-Ra-01

Commit message: Added wide board pcb
Parts:
- U1: footprint lora_tracker:esp32 devkit -> lora_tracker:esp32-devkit-wide
Changed lines of the file:
@@
 EESchema Schematic File Version 4
-LIBS:lora_tracker-cache
-EELAYER 26 0
+EELAYER 30 0
 EELAYER END
 $Descr A4 11693 8268
@@
 F 0 "U1" H 2725 2015 50  0000 C CNN
 F 1 "ESP32" H 2725 1924 50  0000 C CNN
-F 2 "lora_tracker:esp32 devkit" H 2700 2000 50  0001 C CNN
+F 2 "lora_tracker:esp32-devkit-wide" H 2700 2000 50  0001 C CNN
 F 3 "" H 2700 2000 50  0001 C CNN
 	1    2650 1850
