File: extras/schematics/lora_tracker.kicad_pcb (KiCad board)
At the start: 2 copper layers, 40 x 95.2 mm, 18 parts, among them J1 Conn_Coaxial, J2 Conn_01x10_Female, J3 Conn_01x12_Female, J4 Conn_01x03_Female, U1 ESP32, U2 E22-400M30S, U3 Ai-Thinker-Ra-01

Commit message: Updated schematics project
Other:
- net class Default removed
