File: extras/schematics/lora_tracker_wide.kicad_pcb (KiCad board)
At the start: 2 copper layers, 40 x 95.2 mm, 18 parts, among them J1 Conn_Coaxial, J2 Conn_01x10_Female, J3 Conn_01x12_Female, J4 Conn_01x03_Female, U1 ESP32, U2 E22-400M30S, U3 Ai-Thinker-Ra-01

Commit message: Updated schematics project
Other:
- net class Default removed

Commit message: Add missing files
Parts:
- moved JP3 2.34 mm to (102.9, 110.5)
- moved JP1 2.29 mm to (102.9, 101.1)
- moved JP2 2.29 mm to (102.9, 105.9)
- moved JP6 2.29 mm to (102.9, 97.0)
- moved JP7 1.70 mm to (85.1, 88.9)
- moved JP8 0.92 mm to (102.9, 134.6)
Routing:
- net 3v3: track 124.1 -> 120.1 mm
- net Net-(JP2-Pad1): track 10.1 -> 6.79 mm
- net Net-(JP3-Pad1): track 7.60 -> 4.85 mm
- net Net-(JP1-Pad1): track 9.93 -> 7.39 mm
- net MISO: track 71.3 -> 73.6 mm
- net Net-(JP1-Pad3): track 10.7 -> 8.40 mm
- net BUSY: track 96.0 -> 94.1 mm
- net SCK: track 72.7 -> 74.1 mm
- net DIO1: track 97.9 -> 99.0 mm
- net Net-(JP8-Pad1): track 4.99 -> 4.19 mm
- net MOSI: track 64.6 -> 63.9 mm
- net GND: vias 183 -> 178
