File: extras/schematics/esp32c3/esp32_loraprs_c3.kicad_pcb (KiCad board)
At the start: 2 copper layers, 100.8 x 30.2 mm, 28 parts, among them J1 Conn_Coaxial, J2 USB_C_Receptacle_USB2.0, SW1 SW_Push, U1 ESP32_C3_SuperMini, U2 E22-400M30S, U3 IP5306

Commit message: Update schematics
Connections:
- U1 pad 4: DIO2 -> unconnected-(U1-Pad4)
- U2 pad 8: DIO2 -> unconnected-(U2-Pad8)
Routing:
- net DIO2: track 74.9 -> 0.00 mm
- net unconnected-(U1-Pad4): track 0.00 -> 1.37 mm
Changed lines of the file:
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@@
   (net 5 "RXEN")
   (net 6 "DIO1")
-  (net 7 "DIO2")
+  (net 7 "unconnected-(U1-Pad4)")
   (net 8 "SCK")
   (net 9 "unconnected-(U1-Pad6)")
@@
   (net 35 "Net-(D3-Pad2)")
   (net 36 "Net-(JP1-Pad2)")
+  (net 37 "unconnected-(U2-Pad8)")
   (footprint "Capacitor_SMD:C_0805_2012Metric_Pad1.18x1.45mm_HandSolder" (layer "F.Cu")
     (at 124.968 65.278 90)
@@
       (net 6 "DIO1") (pinfunction "GPIO2") (pintype "bidirectional") (solder_mask_margin 0.1016))
     (pad "4" smd rect (at -8.255 15.24 180) (size 1.7 2.5) (layers "F.Cu" "F.Paste" "F.Mask")
-      (net 7 "DIO2") (pinfunction "GPIO3") (pintype "bidirectional") (solder_mask_margin 0.1016))
+      (net 7 "unconnected-(U1-Pad4)") (pinfunction "GPIO3") (pintype "bidirectional+no_connect") (solder_mask_margin 0.1016))
     (pad "5" smd rect (at -8.255 17.78 180) (size 1.7 2.5) (layers "F.Cu" "F.Paste" "F.Mask")
       (net 8 "SCK") (pinfunction "GPIO4") (pintype "bidirectional") (solder_mask_margin 0.1016))
@@
       (net 18 "TXEN") (pinfunction "TXEN") (pintype "bidirectional") (solder_mask_margin 0.1016))
     (pad "8" smd rect locked (at -12 9.05 180) (size 1.7 2.5) (layers "F.Cu" "F.Paste" "F.Mask")
-      (net 7 "DIO2") (pinfunction "DIO2") (pintype "bidirectional") (solder_mask_margin 0.1016))
+      (net 37 "unconnected-(U2-Pad8)") (pinfunction "DIO2") (pintype "bidirectional+no_connect") (solder_mask_margin 0.1016))
     (pad "9" smd rect locked (at -12 11.59 180) (size 1.7 2.5) (layers "F.Cu" "F.Paste" "F.Mask")
       (net 3 "+5V") (pinfunction "VCC@1") (pintype "power_in") (solder_mask_margin 0.1016))
@@
   (via (at 104.14 60.96) (size 0.8) (drill 0.4) (layers "F.Cu" "B.Cu") (net 6))
   (segment (start 104.14 60.96) (end 109.728 66.548) (width 0.2) (layer "B.Cu") (net 6))
-  (segment (start 139.446 67.818) (end 143.764 67.818) (width 0.2) (layer "F.Cu") (net 7))
-  (segment (start 98.966 76.04) (end 114.808 60.198) (width 0.2) (layer "F.Cu") (net 7))
-  (segment (start 143.764 67.818) (end 152.9395 76.9935) (width 0.2) (layer "F.Cu") (net 7))
-  (segment (start 131.826 60.198) (end 139.446 67.818) (width 0.2) (layer "F.Cu") (net 7))
-  (segment (start 98.966 82.104) (end 98.966 76.04) (width 0.2) (layer "F.Cu") (net 7))
   (segment (start 152.9395 76.9935) (end 152.9395 78.359) (width 0.2) (layer "F.Cu") (net 7))
-  (segment (start 114.808 60.198) (end 131.826 60.198) (width 0.2) (layer "F.Cu") (net 7))
   (segment (start 155.4795 75.49555) (end 155.4795 78.359) (width 0.2) (layer "F.Cu") (net 8))
   (segment (start 100.33 72.644) (end 103.632 69.342) (width 0.2) (layer "F.Cu") (net 8))

Commit message: Update schematics
Connections:
- U1 pad 13: BUSY -> unconnected-(U1-Pad13)
- U1 pad 14: unconnected-(U1-Pad14) -> BUSY
- U1 pad 3: DIO1 -> unconnected-(U1-Pad3)
- U1 pad 4: unconnected-(U1-Pad4) -> DIO1
Routing:
- net BUSY: track 57.6 -> 55.0 mm
- net DIO1: track 62.6 -> 65.1 mm
- net unconnected-(U1-Pad4): track 1.37 -> 0.00 mm

Commit message: Added DIP switch for battery
Parts:
- added SW2: SW_DIP_x01, Button_Switch_SMD:SW_SPST_REED_CT05-XXXX-J1, F.Cu at (140.2, 83.3)
- moved R2 6.60 mm to (151.6, 81.8)
- moved R1 6.10 mm to (147.1, 81.8)
Connections:
- C9 pad 1: B+ -> BS+
- L1 pad 2: B+ -> BS+
- R1 pad 1: B+ -> BS+
- R5 pad 1: B+ -> BS+
Routing:
- net BS+: track 0.00 -> 31.3 mm, vias 0 -> 2
- net B+: track 41.9 -> 24.9 mm
- net BS: track 6.36 -> 8.15 mm
- net GND: vias 65 -> 60
